Commit message: update_TA_src_code

File: ROS_H/src/turtlebot3_description/urdf/turtlebot3_waffle.urdf.xacro (robot description, xacro)
@@ -78,6 +78,6 @@
     <origin xyz="0.0 0.154 -0.01" rpy="0 0 0"/>
     <axis xyz="0 0 1"/>
-    <limit lower="-0.02" upper="0" effort="4" velocity="0.5"/>
-    <dynamics damping="0.6" friction="0.3"/>
+    <limit lower="-0.04" upper="0" effort="1000" velocity="1000"/>
+    <dynamics damping="0.0" friction="0.0"/>
   </joint>
   <link name="left_suspension_link">
@@ -129,6 +129,6 @@
     <origin xyz="0.0 -0.154 -0.01" rpy="0 0 0"/>
     <axis xyz="0 0 1"/>
-    <limit lower="-0.02" upper="0" effort="4" velocity="0.5"/>
-    <dynamics damping="0.6" friction="0.3"/>
+    <limit lower="-0.04" upper="0" effort="1000" velocity="1000"/>
+    <dynamics damping="0.0" friction="0.0"/>
   </joint>
   <link name="right_suspension_link">
@@ -180,6 +180,6 @@
     <origin xyz="-0.177 0.064 -0.02" rpy="0 0 0"/>
     <axis xyz="0 0 1"/>
-    <limit lower="-0.01" upper="0" effort="4" velocity="0.5"/>
-    <dynamics damping="0.6" friction="0.3"/>
+    <limit lower="-0.04" upper="0" effort="1000" velocity="1000"/>
+    <dynamics damping="0.0" friction="0.0"/>
   </joint>
   <link name="left_caster_link">
@@ -190,4 +190,10 @@
       </geometry>
     </collision>
+    <visual>
+      <origin xyz="0 0.001 0" rpy="-1.57 0 0"/>
+      <geometry>
+        <sphere radius="0.02"/>
+      </geometry>
+    </visual>
     <inertial>
       <origin xyz="0 0 0" />
@@ -203,6 +209,6 @@
     <origin xyz="-0.177 -0.064 -0.02" rpy="0 0 0"/>
     <axis xyz="0 0 1"/>
-    <limit lower="-0.01" upper="0" effort="4" velocity="0.5"/>
-    <dynamics damping="0.6" friction="0.3"/>
+    <limit lower="-0.04" upper="0" effort="1000" velocity="1000"/>
+    <dynamics damping="0.0" friction="0.0"/>
   </joint>
   <link name="right_caster_link">
@@ -213,4 +219,10 @@
       </geometry>
     </collision>
+    <visual>
+      <origin xyz="0 0.001 0" rpy="-1.57 0 0"/>
+      <geometry>
+        <sphere radius="0.02"/>
+      </geometry>
+    </visual>
     <inertial>
       <origin xyz="0 0 0" />
