Commit message: lidar_cam_functioning_and_speed_increased

File: ROS/packages_sample/toy_car/urdf/toy_car2.urdf (robot description, URDF)
Before this commit: robot toy_car, 7 links, 6 joints
Links:
- added link camera_center, mass 0.043612; collision mesh filename=package://toy_car/meshes/camera_center.STL; visual mesh filename=package://toy_car/meshes/camera_center.STL
- added link camera_left, mass 0.043612; collision mesh filename=package://toy_car/meshes/camera_left.STL; visual mesh filename=package://toy_car/meshes/camera_left.STL
- added link camera_right, mass 0.0436119950287126; collision mesh filename=package://toy_car/meshes/camera_right.STL; visual mesh filename=package://toy_car/meshes/camera_right.STL
- added link lidar_top, mass 0.073085; collision mesh filename=package://toy_car/meshes/lidar_top.STL; visual mesh filename=package://toy_car/meshes/lidar_top.STL
- link base_link: mass 3.0763 -> 3.4415
- link front_left_wheel: mass 0.8936 -> 0.389
- link front_right_wheel: mass 0.8936 -> 0.389
- link rear_left_caster: mass 0.017712 -> 0.0175
- link rear_left_caster_wheel: mass 0.025494 -> 0.025328
- link rear_right_caster: mass 0.017712 -> 0.0175
- link rear_right_caster_wheel: mass 0.025494 -> 0.025328
Joints:
- added joint camera_center_joint: type fixed, parent base_link, child camera_center, origin xyz=-0.072595 -0.15 0.128 rpy=0 0.2012 -3.1416, axis 0 0 0
- added joint camera_left_joint: type fixed, parent base_link, child camera_left, origin xyz=-0.0375 -0.275 0.134 rpy=0 0 -3.1416, axis 0 0 0
- added joint camera_right_joint: type fixed, parent base_link, child camera_right, origin xyz=-0.0375 -0.025 0.134 rpy=0 0 3.1416, axis 0 0 0
- added joint lidar_top_joint: type fixed, parent base_link, child lidar_top, origin xyz=0.081303 -0.15 0.1865 rpy=0 0 0, axis 0 0 0
- joint front_left_wheel_joint: limit effort=2.3 velocity=5.23 -> effort=3.1 velocity=7; origin xyz=1.2819E-05 -0.3265 -0.003 rpy=1.5708 0.86221 0 -> xyz=1.2819E-05 -0.3265 -0.003 rpy=1.5708 0 0
- joint front_right_wheel_joint: limit effort=2.3 velocity=5.23 -> effort=3.1 velocity=7; origin xyz=-1.2819E-05 0.0265 -0.003 rpy=1.5708 -0.067638 0 -> xyz=-1.2819E-05 0.0265 -0.003 rpy=1.5708 0 0
- joint rear_left_caster_joint: limit (none) -> lower=0 upper=0 effort=0 velocity=0; origin xyz=0.22 -0.26 -0.0225 rpy=1.5708 0 3.0462 -> xyz=0.22 -0.26 -0.0235 rpy=1.5708 0 0
- joint rear_left_caster_wheel_joint: origin xyz=-0.008 -0.033 0 rpy=-3.1416 0 -2.9205 -> xyz=0.008 -0.032 0 rpy=0 0 -0.21884
- joint rear_right_caster_joint: limit (none) -> lower=0 upper=0 effort=0 velocity=0; origin xyz=0.22 -0.04 -0.0225 rpy=1.5708 0 3.078 -> xyz=0.22 -0.04 -0.0235 rpy=1.5708 0 0
- joint rear_right_caster_wheel_joint: origin xyz=-0.008 -0.033 0 rpy=0 0 -0.38747 -> xyz=0.008 -0.032 0 rpy=3.1416 0 0.10137

Commit message: new_car_with_suspension

File: ROS/packages_sample/toy_car/urdf/toy_car2.urdf (robot description, URDF)
Before this commit: robot toy_car, 11 links, 10 joints
Links:
- removed link camera_center
- removed link camera_left
- removed link camera_right
- removed link lidar_top
- removed link rear_left_caster
- removed link rear_left_caster_wheel
- removed link rear_right_caster
- removed link rear_right_caster_wheel
- added link cam_center, mass 0.0436119958195422; collision mesh filename=package://toy_car/meshes/cam_center.STL; visual mesh filename=package://toy_car/meshes/cam_center.STL
- added link cam_left, mass 0.0436119950287128; collision mesh filename=package://toy_car/meshes/cam_left.STL; visual mesh filename=package://toy_car/meshes/cam_left.STL
- added link cam_right, mass 0.0436119950287128; collision mesh filename=package://toy_car/meshes/cam_right.STL; visual mesh filename=package://toy_car/meshes/cam_right.STL
- added link dummy, mass 0.001; collision mesh filename=package://toy_car/meshes/dummy.STL; visual mesh filename=package://toy_car/meshes/dummy.STL
- added link front_left, mass 0.0211105794692306; collision mesh filename=package://toy_car/meshes/front_left.STL; visual mesh filename=package://toy_car/meshes/front_left.STL
- added link front_left_suspension, mass 0.108487939485068; collision mesh filename=package://toy_car/meshes/front_left_suspension.STL; visual mesh filename=package://toy_car/meshes/front_left_suspension.STL
- added link front_right, mass 0.0211105794692306; collision mesh filename=package://toy_car/meshes/front_right.STL; visual mesh filename=package://toy_car/meshes/front_right.STL
- added link front_right_suspension, mass 0.108487939485068; collision mesh filename=package://toy_car/meshes/front_right_suspension.STL; visual mesh filename=package://toy_car/meshes/front_right_suspension.STL
- added link imu, mass 0.000999999999999999; collision mesh filename=package://toy_car/meshes/imu.STL; visual mesh filename=package://toy_car/meshes/imu.STL
- added link lidar, mass 0.0730845703017379; collision mesh filename=package://toy_car/meshes/lidar.STL; visual mesh filename=package://toy_car/meshes/lidar.STL
- added link rear_left, mass 0.00600385822447067; collision mesh filename=package://toy_car/meshes/rear_left.STL; visual mesh filename=package://toy_car/meshes/rear_left.STL
- added link rear_left_suspension, mass 0.0815242305195134; collision mesh filename=package://toy_car/meshes/rear_left_suspension.STL; visual mesh filename=package://toy_car/meshes/rear_left_suspension.STL
- added link rear_right, mass 0.00600385822447067; collision mesh filename=package://toy_car/meshes/rear_right.STL; visual mesh filename=package://toy_car/meshes/rear_right.STL
- added link rear_right_suspension, mass 0.0815242305195134; collision mesh filename=package://toy_car/meshes/rear_right_suspension.STL; visual mesh filename=package://toy_car/meshes/rear_right_suspension.STL
- link base_link: mass 3.4415 -> 3.81368362259093
- link front_left_wheel: mass 0.389 -> 0.389004584885854
- link front_right_wheel: mass 0.389 -> 0.389004584885853
Joints:
- removed joint camera_center_joint
- removed joint camera_left_joint
- removed joint camera_right_joint
- removed joint lidar_top_joint
- removed joint rear_left_caster_joint
- removed joint rear_left_caster_wheel_joint
- removed joint rear_right_caster_joint
- removed joint rear_right_caster_wheel_joint
- added joint cam_center_joint: type fixed, parent base_link, child cam_center, origin xyz=0.065337 0 0.1132 rpy=0 0.2012 0, axis 0 0 0
- added joint cam_left_joint: type fixed, parent base_link, child cam_left, origin xyz=0.0245 0.125 0.11 rpy=0 0 0, axis 0 0 0
- added joint cam_right_joint: type fixed, parent base_link, child cam_right, origin xyz=0.0245 -0.125 0.10999737041193 rpy=0 0 0, axis 0 0 0
- added joint dummy_joint: type fixed, parent base_link, child dummy, origin xyz=-0.005 0 0.135 rpy=0 0 0, axis 0 0 0
- added joint front_left_joint: type fixed, parent base_link, child front_left, origin xyz=-0.021 0.125 0.11499737041193 rpy=0 0 0, axis 0 0 0
- added joint front_left_suspension_joint: type prismatic, parent front_left, child front_left_suspension, origin xyz=0 0.0273428886495924 -0.07 rpy=0.17453292519943 0 0, axis 0 0 -1, limit lower=-0.03 upper=0.03 effort=1000 velocity=1000
- added joint front_right_joint: type fixed, parent base_link, child front_right, origin xyz=-0.0210000000000001 -0.125 0.11499737041193 rpy=0 0 0, axis 0 0 0
- added joint front_right_suspension_joint: type prismatic, parent front_right, child front_right_suspension, origin xyz=0 -0.0273428886495923 -0.07 rpy=-0.17453292519943 0 0, axis 0 0 -1, limit lower=-0.03 upper=0.03 effort=1000 velocity=1000
- added joint imu_joint: type fixed, parent base_link, child imu, origin xyz=-0.00499999999999977 0 0.13499737041193 rpy=0 0 0, axis 0 0 0
- added joint lidar_joint: type fixed, parent base_link, child lidar, origin xyz=-0.085232 0 0.177 rpy=0 0 0, axis 0 0 0
- added joint rear_left_joint: type fixed, parent base_link, child rear_left, origin xyz=-0.288495633593833 0.1025 0.0564000000000001 rpy=0 0 0, axis 0 0 0
- added joint rear_left_suspension_joint: type prismatic, parent rear_left, child rear_left_suspension, origin xyz=0 0 -0.06 rpy=0 0 0, axis 0 0 -1, limit lower=-0.02 upper=0.02 effort=1000 velocity=1000
- added joint rear_right: type fixed, parent base_link, child rear_right, origin xyz=-0.288495633593834 -0.1025 0.0564000000000001 rpy=0 0 0, axis 0 0 0
- added joint rear_right_suspension_joint: type prismatic, parent rear_right, child rear_right_suspension, origin xyz=0 0 -0.06 rpy=0 0 0, axis 0 0 -1, limit lower=-0.02 upper=0.02 effort=1000 velocity=1000
- joint front_left_wheel_joint: axis 0 0 1 -> 0 1 0; origin xyz=1.2819E-05 -0.3265 -0.003 rpy=1.5708 0 0 -> xyz=1.12457305640069E-05 0.0310624201259151 -0.0649811422108027 rpy=-0.17453292519943 0 0; parent base_link -> front_left_suspension
- joint front_right_wheel_joint: axis 0 0 1 -> 0 1 0; origin xyz=-1.2819E-05 0.0265 -0.003 rpy=1.5708 0 0 -> xyz=-1.1246E-05 -0.031062 -0.064981 rpy=0.17453 0 0; parent base_link -> front_right_suspension

Commit message: new_model_camera_lidar

File: ROS/packages_sample/toy_car/urdf/toy_car2.urdf (robot description, URDF)
Before this commit: robot toy_car2, 17 links, 16 joints
Links:
- removed link cam_center
- removed link cam_left
- removed link cam_right
- removed link lidar
- added link camera_center, mass 0.0436119958195422; collision mesh filename=package://toy_car/meshes/cam_center.STL; visual mesh filename=package://toy_car/meshes/cam_center.STL
- added link camera_left, mass 0.0436119950287128; collision mesh filename=package://toy_car/meshes/cam_left.STL; visual mesh filename=package://toy_car/meshes/cam_left.STL
- added link camera_right, mass 0.0436119950287128; collision mesh filename=package://toy_car/meshes/cam_right.STL; visual mesh filename=package://toy_car/meshes/cam_right.STL
- added link lidar_top, mass 0.0730845703017379; collision mesh filename=package://toy_car/meshes/lidar.STL; visual mesh filename=package://toy_car/meshes/lidar.STL
Joints:
- removed joint cam_center_joint
- removed joint cam_left_joint
- removed joint cam_right_joint
- added joint camera_center_joint: type fixed, parent base_link, child camera_center, origin xyz=0.065337 0 0.1132 rpy=0 0.2012 0, axis 0 0 0
- added joint camera_left_joint: type fixed, parent base_link, child camera_left, origin xyz=0.0245 0.125 0.11 rpy=0 0 0, axis 0 0 0
- added joint camera_right_joint: type fixed, parent base_link, child camera_right, origin xyz=0.0245 -0.125 0.10999737041193 rpy=0 0 0, axis 0 0 0
- joint lidar_joint: child lidar -> lidar_top

Commit message: newmodel

File: ROS/packages_sample/toy_car/urdf/toy_car2.urdf (robot description, URDF)
Before this commit: robot toy_car2, 17 links, 16 joints
Links:
- added link camera_link, mass 0.056857; collision mesh filename=package://toy_car/meshes/camera_link.STL; visual mesh filename=package://toy_car/meshes/camera_link.STL
- added link holder, mass 1.432834; collision mesh filename=package://toy_car/meshes/holder.STL; visual mesh filename=package://toy_car/meshes/holder.STL
- added link jetson, mass 0.2; collision mesh filename=package://toy_car/meshes/jetson.STL; visual mesh filename=package://toy_car/meshes/jetson.STL
- added link nuc, mass 0.39954; collision mesh filename=package://toy_car/meshes/nuc.STL; visual mesh filename=package://toy_car/meshes/nuc.STL
- added link rio, mass 0.193; collision mesh filename=package://toy_car/meshes/rio.STL; visual mesh filename=package://toy_car/meshes/rio.STL
- link base_link: mass 3.81368362259093 -> 1.44712978241803
- link camera_center: mass 0.0436119958195422 -> 0.061453; geometry collision mesh filename=package://toy_car/meshes/camera_center.STL; visual mesh filename=package://toy_car/meshes/camera_center.STL
- link camera_left: mass 0.0436119950287128 -> 0.061453; geometry collision mesh filename=package://toy_car/meshes/camera_left.STL; visual mesh filename=package://toy_car/meshes/camera_left.STL
- link camera_right: mass 0.0436119950287128 -> 0.061453; geometry collision mesh filename=package://toy_car/meshes/camera_right.STL; visual mesh filename=package://toy_car/meshes/camera_right.STL
- link dummy: mass 0.001 -> 0
- link front_left_wheel: mass 0.389004584885854 -> 0.389004584885853
- link front_right_suspension: mass 0.108487939485068 -> 0.108487813658331
- link imu: mass 0.000999999999999999 -> 0.001
- link lidar_top: mass 0.0730845703017379 -> 0.2; geometry collision mesh filename=package://toy_car/meshes/lidar_top.STL; visual mesh filename=package://toy_car/meshes/lidar_top.STL
- link rear_left_suspension: mass 0.0815242305195134 -> 0.0912015925296314
- link rear_right_suspension: mass 0.0815242305195134 -> 0.0912015925296314
Joints:
- removed joint lidar_joint
- removed joint rear_right
- added joint camera_link_joint: type fixed, parent base_link, child camera_link, origin xyz=0.027007 0 0.105 rpy=0 0 0, axis 0 0 0
- added joint holder_joint: type fixed, parent base_link, child holder, origin xyz=0.0015 0 0.019999 rpy=0 0 0, axis 0 0 0
- added joint jetson_joint: type fixed, parent base_link, child jetson, origin xyz=-0.1085 0 0.0671 rpy=0 0 0, axis 0 0 0
- added joint lidar_top_joint: type fixed, parent base_link, child lidar_top, origin xyz=-0.085232 0 0.177 rpy=0 0 0, axis 0 0 0
- added joint nuc_joint: type fixed, parent base_link, child nuc, origin xyz=-0.073998 7.38E-05 0.0071 rpy=0 0 0, axis 0 0 0
- added joint rear_right_joint: type fixed, parent base_link, child rear_right, origin xyz=-0.2885 -0.1025 0.0564 rpy=0 0 0, axis 0 0 0
- added joint rio_joint: type fixed, parent base_link, child rio, origin xyz=-0.062748 0 0.0391 rpy=0 0 0, axis 0 0 0
- joint camera_center_joint: origin xyz=0.065337 0 0.1132 rpy=0 0.2012 0 -> xyz=0.0383297438164813 0 0.00819952580620682 rpy=0 0.201198652587711 0; parent base_link -> camera_link
- joint camera_right_joint: origin xyz=0.0245 -0.125 0.10999737041193 rpy=0 0 0 -> xyz=0.0245 -0.125 0.11 rpy=0 0 0
- joint dummy_joint: origin xyz=-0.005 0 0.135 rpy=0 0 0 -> xyz=-0.00499999999999977 0 0.13499737041193 rpy=0 0 0
- joint front_left_suspension_joint: limit lower=-0.03 upper=0.03 effort=1000 velocity=1000 -> lower=-0.03 upper=0.03 effort=30 velocity=100
- joint front_right_joint: origin xyz=-0.0210000000000001 -0.125 0.11499737041193 rpy=0 0 0 -> xyz=-0.021 -0.125 0.11499737041193 rpy=0 0 0
- joint front_right_suspension_joint: limit lower=-0.03 upper=0.03 effort=1000 velocity=1000 -> lower=-0.03 upper=0.03 effort=30 velocity=100
- joint front_right_wheel_joint: origin xyz=-1.1246E-05 -0.031062 -0.064981 rpy=0.17453 0 0 -> xyz=1.1246E-05 -0.031062 -0.064981 rpy=0.17453 0 0
- joint imu_joint: origin xyz=-0.00499999999999977 0 0.13499737041193 rpy=0 0 0 -> xyz=-0.005 0 0.135 rpy=0 0 0
- joint rear_left_joint: origin xyz=-0.288495633593833 0.1025 0.0564000000000001 rpy=0 0 0 -> xyz=-0.2885 0.1025 0.0564 rpy=0 0 0
- joint rear_left_suspension_joint: limit lower=-0.02 upper=0.02 effort=1000 velocity=1000 -> lower=-0.02 upper=0.02 effort=30 velocity=100
- joint rear_right_suspension_joint: limit lower=-0.02 upper=0.02 effort=1000 velocity=1000 -> lower=-0.02 upper=0.02 effort=30 velocity=100

Commit message: new_model_holder_stuck_improved

File: ROS/packages_sample/toy_car/urdf/toy_car2.urdf (robot description, URDF)
Before this commit: robot toy_car2, 22 links, 21 joints
Links:
- added link left_plate, mass 0.001455; collision mesh filename=package://toy_car/meshes/left_plate.STL; visual mesh filename=package://toy_car/meshes/left_plate.STL
- added link right_plate, mass 0.001455; collision mesh filename=package://toy_car/meshes/right_plate.STL; visual mesh filename=package://toy_car/meshes/right_plate.STL
- link base_link: mass 1.44712978241803 -> 1.4471
- link front_left: mass 0.0211105794692306 -> 0.021111
- link front_left_suspension: mass 0.108487939485068 -> 0.10849
- link front_left_wheel: mass 0.389004584885853 -> 0.389
- link front_right_suspension: mass 0.108487813658331 -> 0.10849
- link front_right_wheel: mass 0.389004584885853 -> 0.389
- link holder: mass 1.432834 -> 1.4328
- link rear_left: mass 0.00600385822447067 -> 0.0060039
- link rear_left_suspension: mass 0.0912015925296314 -> 0.091202
- link rear_right: mass 0.00600385822447067 -> 0.0060039
- link rear_right_suspension: mass 0.0912015925296314 -> 0.091202
- link rio: mass 0.193 -> 0.192
Joints:
- added joint left_plate_joint: type fixed, parent holder, child left_plate, origin xyz=0.12963 0.0875 -0.02548 rpy=0 0.50284 0, axis 0 0 0
- added joint right_plate_joint: type fixed, parent holder, child right_plate, origin xyz=0.12963 -0.0875 -0.02548 rpy=0 0.50284 0, axis 0 0 0
- joint camera_center_joint: origin xyz=0.0383297438164813 0 0.00819952580620682 rpy=0 0.201198652587711 0 -> xyz=0.0404208856688172 0 0.0046602540378443 rpy=0 0.523598775598297 0
- joint dummy_joint: origin xyz=-0.00499999999999977 0 0.13499737041193 rpy=0 0 0 -> xyz=-0.005 0 0.135 rpy=0 0 0
- joint front_left_joint: origin xyz=-0.021 0.125 0.11499737041193 rpy=0 0 0 -> xyz=-0.021 0.125 0.115 rpy=0 0 0
- joint front_left_suspension_joint: origin xyz=0 0.0273428886495924 -0.07 rpy=0.17453292519943 0 0 -> xyz=0 0.027343 -0.07 rpy=0.17453 0 0
- joint front_left_wheel_joint: origin xyz=1.12457305640069E-05 0.0310624201259151 -0.0649811422108027 rpy=-0.17453292519943 0 0 -> xyz=1.1246E-05 0.031062 -0.064981 rpy=-0.17453 0 0
- joint front_right_joint: origin xyz=-0.021 -0.125 0.11499737041193 rpy=0 0 0 -> xyz=-0.021 -0.125 0.115 rpy=0 0 0
- joint front_right_suspension_joint: origin xyz=0 -0.0273428886495923 -0.07 rpy=-0.17453292519943 0 0 -> xyz=0 -0.027343 -0.07 rpy=-0.17453 0 0
- joint holder_joint: origin xyz=0.0015 0 0.019999 rpy=0 0 0 -> xyz=0.0015 0 0.034999 rpy=0 0 0
- joint imu_joint: origin xyz=-0.005 0 0.135 rpy=0 0 0 -> xyz=-0.00499999999999977 0 0.13499737041193 rpy=0 0 0
- joint rear_left_joint: origin xyz=-0.2885 0.1025 0.0564 rpy=0 0 0 -> xyz=-0.288495633593833 0.1025 0.0564000000000001 rpy=0 0 0
